Commit message: Add to xacro file the definition for the links for each wheel Add to xacro file the definition for the joints for each wheel

File: urdf/udacity_bot.xacro (robot description, xacro)
@@ -55,3 +55,67 @@
     </visual>
   </link>
+<joint type="continuous" name="left_wheel_hinge">
+    <origin xyz="0 0.15 0" rpy="0 0 0"/>
+    <child link="left_wheel"/>
+    <parent link="chassis"/>
+    <axis xyz="0 1 0" rpy="0 0 0"/>
+    <limit effort="10000" velocity="1000"/>
+    <dynamics damping="1.0" friction="1.0"/>
+  </joint>
+<link name='left_wheel'>
+    <pose>0 0 0.1 0 0 0</pose>
+    <inertial>
+      <mass value="5.0"/>
+      <origin xyz="0.0 0 0" rpy=" 0 1.5707 1.5707"/>
+      <inertia
+          ixx="0.1" ixy="0" ixz="0"
+          iyy="0.1" iyz="0"
+          izz="0.1"
+      />
+    </inertial>
+    <collision name='left_wheel_collision'>
+      <origin xyz="0.0 0 0" rpy=" 0 1.5707 1.5707"/>
+      <geometry>
+        <cylinder radius="0.1" length="0.05"/>
+      </geometry>
+    </collision>
+    <visual name='left_wheel_visual'>
+      <origin xyz="0.0 0 0" rpy=" 0 1.5707 1.5707"/>
+      <geometry>
+        <cylinder radius="0.1" length="0.05"/>
+      </geometry>
+    </visual>
+  </link>
+<joint type="continuous" name="right_wheel_hinge">
+    <origin xyz="0 -0.15 0" rpy="0 0 0"/>
+    <child link="right_wheel"/>
+    <parent link="chassis"/>
+    <axis xyz="0 1 0" rpy="0 0 0"/>
+    <limit effort="10000" velocity="1000"/>
+    <dynamics damping="1.0" friction="1.0"/>
+  </joint>
+<link name='right_wheel'>
+    <pose>0 0 0.1 0 0 0</pose>
+    <inertial>
+      <mass value="5.0"/>
+      <origin xyz="0.0 0 0" rpy=" 0 1.5707 1.5707"/>
+      <inertia
+          ixx="0.1" ixy="0" ixz="0"
+          iyy="0.1" iyz="0"
+          izz="0.1"
+      />
+    </inertial>
+    <collision name='right_wheel_collision'>
+      <origin xyz="0.0 0 0" rpy=" 0 1.5707 1.5707"/>
+      <geometry>
+        <cylinder radius="0.1" length="0.05"/>
+      </geometry>
+    </collision>
+    <visual name='right_wheel_visual'>
+      <origin xyz="0.0 0 0" rpy=" 0 1.5707 1.5707"/>
+      <geometry>
+        <cylinder radius="0.1" length="0.05"/>
+      </geometry>
+    </visual>
+  </link>
 </robot>

Commit message: Add to xacro file the camera (definition for the link and joint)

File: urdf/udacity_bot.xacro (robot description, xacro)
@@ -119,3 +119,33 @@
     </visual>
   </link>
+<!-- Camera -->
+<link name="camera">
+    <pose>0 0 0.1 0 0 0</pose>
+    <inertial>
+      <mass value="0.1"/>
+      <origin xyz="0.0 0 0" rpy="0 0 0"/>
+      <inertia
+          ixx="0.0001" ixy="0" ixz="0"
+          iyy="0.0001" iyz="0"
+          izz="0.0001"
+      />
+    </inertial>
+    <collision name='camera_collision'>
+      <origin xyz="0.0 0 0" rpy="0 0 0"/>
+      <geometry>
+        <box size="0.05 0.05 0.05"/>
+      </geometry>
+    </collision>
+    <visual name='camera_visual'>
+      <origin xyz="0.0 0 0" rpy="0 0 0"/>
+      <geometry>
+         <box size="0.05 0.05 0.05"/>
+      </geometry>
+    </visual>
+  </link>
+<joint type="fixed" name="camera_joint">
+    <origin xyz="0.2 0 0" rpy="0 0 0"/>
+    <child link="camera"/>
+    <parent link="chassis"/>
+  </joint>
 </robot>

Commit message: Add to xacro file the hokuyo laser (definition for the link (as a box) and joint)

File: urdf/udacity_bot.xacro (robot description, xacro)
@@ -149,3 +149,33 @@
     <parent link="chassis"/>
   </joint>
+<!-- Laser -->
+<link name="hokuyo">
+    <pose>0 0 0.1 0 0 0</pose>
+    <inertial>
+      <mass value="0.1"/>
+      <origin xyz="0.0 0 0" rpy="0 0 0"/>
+      <inertia
+          ixx="0.0001" ixy="0" ixz="0"
+          iyy="0.0001" iyz="0"
+          izz="0.0001"
+      />
+    </inertial>
+    <collision name='hokuyo_collision'>
+      <origin xyz="0.0 0 0" rpy="0 0 0"/>
+      <geometry>
+        <box size="0.1 0.1 0.1"/>
+      </geometry>
+    </collision>
+    <visual name='hokuyo_visual'>
+      <origin xyz="0.0 0 0" rpy="0 0 0"/>
+      <geometry>
+         <box size="0.1 0.1 0.1"/>
+      </geometry>
+    </visual>
+  </link>
+<joint type="fixed" name="hokuyo_joint">
+    <origin xyz="0.15 0 0.1" rpy="0 0 0"/>
+    <child link="hokuyo"/>
+    <parent link="chassis"/>
+  </joint>
 </robot>

Commit message: Edit xacro file, hokuyo laser: change visual geometry to mesh file

File: urdf/udacity_bot.xacro (robot description, xacro)
@@ -170,5 +170,5 @@
       <origin xyz="0.0 0 0" rpy="0 0 0"/>
       <geometry>
-         <box size="0.1 0.1 0.1"/>
+         <mesh filename="package://udacity_bot/meshes/hokuyo.dae"/>
       </geometry>
     </visual>

Commit message: Edit robot model: increase chassis height, elevate camera position

File: urdf/udacity_bot.xacro (robot description, xacro)
@@ -4,10 +4,10 @@
   <link name="robot_footprint"></link>
   <joint name="robot_footprint_joint" type="fixed">
-    <origin xyz="0 0 0" rpy="0 0 0" />
+    <origin xyz="0 0 0.12" rpy="0 0 0" />
     <parent link="robot_footprint"/>
     <child link="chassis" />
   </joint>
   <link name='chassis'>
-    <pose>0 0 0.1 0 0 0</pose>
+    <pose>0 0 0 0 0 0</pose>
     <inertial>
       <mass value="15.0"/>
@@ -22,5 +22,5 @@
       <origin xyz="0 0 0" rpy=" 0 0 0"/>
       <geometry>
-        <box size=".4 .2 .1"/>
+        <box size=".4 .2 .12"/>
       </geometry>
     </collision>
@@ -28,9 +28,9 @@
       <origin xyz="0 0 0" rpy=" 0 0 0"/>
       <geometry>
-        <box size=".4 .2 .1"/>
+        <box size=".4 .2 .12"/>
       </geometry>
     </visual>
     <collision name='back_caster_collision'>
-      <origin xyz="-0.15 0 -0.05" rpy=" 0 0 0"/>
+      <origin xyz="-0.15 0 -0.1" rpy=" 0 0 0"/>
       <geometry>
         <sphere radius="0.0499"/>
@@ -38,5 +38,5 @@
     </collision>
     <visual name='back_caster_visual'>
-      <origin xyz="-0.15 0 -0.05" rpy=" 0 0 0"/>
+      <origin xyz="-0.15 0 -0.1" rpy=" 0 0 0"/>
       <geometry>
         <sphere radius="0.05"/>
@@ -44,5 +44,5 @@
     </visual>
     <collision name='front_caster_collision'>
-      <origin xyz="0.15 0 -0.05" rpy=" 0 0 0"/>
+      <origin xyz="0.15 0 -0.1" rpy=" 0 0 0"/>
       <geometry>
         <sphere radius="0.0499"/>
@@ -50,5 +50,5 @@
     </collision>
     <visual name='front_caster_visual'>
-      <origin xyz="0.15 0 -0.05" rpy=" 0 0 0"/>
+      <origin xyz="0.15 0 -0.1" rpy=" 0 0 0"/>
       <geometry>
         <sphere radius="0.05"/>
@@ -57,5 +57,5 @@
   </link>
 <joint type="continuous" name="left_wheel_hinge">
-    <origin xyz="0 0.15 0" rpy="0 0 0"/>
+    <origin xyz="0 0.15 -0.05" rpy="0 0 0"/>
     <child link="left_wheel"/>
     <parent link="chassis"/>
@@ -76,5 +76,5 @@
     </inertial>
     <collision name='left_wheel_collision'>
-      <origin xyz="0.0 0 0" rpy=" 0 1.5707 1.5707"/>
+      <origin xyz="0 0 0" rpy=" 0 1.5707 1.5707"/>
       <geometry>
         <cylinder radius="0.1" length="0.05"/>
@@ -89,5 +89,5 @@
   </link>
 <joint type="continuous" name="right_wheel_hinge">
-    <origin xyz="0 -0.15 0" rpy="0 0 0"/>
+    <origin xyz="0 -0.15 -0.05" rpy="0 0 0"/>
     <child link="right_wheel"/>
     <parent link="chassis"/>
@@ -122,5 +122,4 @@
 <!-- Camera -->
 <link name="camera">
-    <pose>0 0 0.1 0 0 0</pose>
     <inertial>
       <mass value="0.1"/>
@@ -135,5 +134,5 @@
       <origin xyz="0.0 0 0" rpy="0 0 0"/>
       <geometry>
-        <box size="0.05 0.05 0.05"/>
+        <box size="0.02 0.05 0.05"/>
       </geometry>
     </collision>
@@ -141,10 +140,10 @@
       <origin xyz="0.0 0 0" rpy="0 0 0"/>
       <geometry>
-         <box size="0.05 0.05 0.05"/>
+         <box size="0.02 0.05 0.05"/>
       </geometry>
     </visual>
   </link>
 <joint type="fixed" name="camera_joint">
-    <origin xyz="0.2 0 0" rpy="0 0 0"/>
+    <origin xyz="0.2 0 0.025" rpy="0 0 0"/>
     <child link="camera"/>
     <parent link="chassis"/>
@@ -176,5 +175,5 @@
   </link>
 <joint type="fixed" name="hokuyo_joint">
-    <origin xyz="0.15 0 0.1" rpy="0 0 0"/>
+    <origin xyz="0.15 0 0.09" rpy="0 0 0"/>
     <child link="hokuyo"/>
     <parent link="chassis"/>

Commit message: Add new camera mesh to robot model

File: urdf/udacity_bot.xacro (robot description, xacro)
@@ -137,4 +137,5 @@
       </geometry>
     </collision>
+<!--
     <visual name='camera_visual'>
       <origin xyz="0.0 0 0" rpy="0 0 0"/>
@@ -143,7 +144,14 @@
       </geometry>
     </visual>
+-->
+    <visual name='camera_visual'>
+      <origin xyz="0 0 0" rpy="0 0 0"/>
+      <geometry>
+         <mesh filename="package://udacity_bot/meshes/camera.dae"/>
+      </geometry>
+    </visual>
   </link>
 <joint type="fixed" name="camera_joint">
-    <origin xyz="0.2 0 0.025" rpy="0 0 0"/>
+    <origin xyz="0.205 0.0 0.07" rpy="0 0 0"/>
     <child link="camera"/>
     <parent link="chassis"/>
@@ -175,5 +183,5 @@
   </link>
 <joint type="fixed" name="hokuyo_joint">
-    <origin xyz="0.15 0 0.09" rpy="0 0 0"/>
+    <origin xyz="0.135 0 0.09" rpy="0 0 0"/> <!-- 0.15 -->
     <child link="hokuyo"/>
     <parent link="chassis"/>

Commit message: Fix regular RGB camera tf frame orientation. Refactor camera .xacro and .gazebo by moving compenents into separate files

File: urdf/udacity_bot.xacro (robot description, xacro)
@@ -7,4 +7,6 @@
 <xacro:arg name="diff_drive_publishTf" default="true" />
 <xacro:arg name="diff_drive_publishOdomTF" default="true" />
+<!-- Determine presence of camera sensor -->
+<xacro:arg name="add_camera_sensor" default="true" />
 <!-- Configure ground truth odometry Gazebo plugin -->
 <xacro:arg name="p3d_base_controller_enabled" default="false" />
@@ -13,4 +15,5 @@
 <xacro:include filename="$(find udacity_bot)/urdf/p3d_base_controller.gazebo" />
 </xacro:if>
+<!-- Determine the name of the robot's root link -->
   <link name="robot_footprint"></link>
   <joint name="robot_footprint_joint" type="fixed">
@@ -131,41 +134,11 @@
     </visual>
   </link>
-<!-- Camera -->
-<link name="camera">
-    <inertial>
-      <mass value="0.1"/>
-      <origin xyz="0.0 0 0" rpy="0 0 0"/>
-      <inertia
-          ixx="0.0001" ixy="0" ixz="0"
-          iyy="0.0001" iyz="0"
-          izz="0.0001"
-      />
-    </inertial>
-    <collision name='camera_collision'>
-      <origin xyz="0.0 0 0" rpy="0 0 0"/>
-      <geometry>
-        <box size="0.02 0.05 0.05"/>
-      </geometry>
-    </collision>
-<!--
-    <visual name='camera_visual'>
-      <origin xyz="0.0 0 0" rpy="0 0 0"/>
-      <geometry>
-         <box size="0.02 0.05 0.05"/>
-      </geometry>
-    </visual>
--->
-    <visual name='camera_visual'>
-      <origin xyz="0 0 0" rpy="0 0 0"/>
-      <geometry>
-         <mesh filename="package://udacity_bot/meshes/camera.dae"/>
-      </geometry>
-    </visual>
-  </link>
-<joint type="fixed" name="camera_joint">
-    <origin xyz="0.205 0.0 0.07" rpy="0 0 0"/>
-    <child link="camera"/>
-    <parent link="chassis"/>
-  </joint>
+<!-- Add a regular RGB Camera -->
+<xacro:if value="$(arg add_camera_sensor)">
+  <!-- Add Camera link, joints and mesh -->
+  <xacro:include filename="$(find udacity_bot)/urdf/rgb_camera.xacro"/>
+  <!-- Add Gazebo Camera Plugin -->
+  <xacro:include filename="$(find udacity_bot)/urdf/rgb_camera.gazebo"/>
+</xacro:if>
 <!-- Laser -->
 <link name="hokuyo">

Commit message: Refactor laser in .xacro and .gazebo files by moving compenents into separate files

File: urdf/udacity_bot.xacro (robot description, xacro)
@@ -7,6 +7,8 @@
 <xacro:arg name="diff_drive_publishTf" default="true" />
 <xacro:arg name="diff_drive_publishOdomTF" default="true" />
-<!-- Determine presence of camera sensor -->
+<!-- Determine presence of RGB camera sensor -->
 <xacro:arg name="add_camera_sensor" default="true" />
+<!-- Determine presence of Hokuyo laser sensor -->
+<xacro:arg name="add_laser_sensor" default="true" />
 <!-- Configure ground truth odometry Gazebo plugin -->
 <xacro:arg name="p3d_base_controller_enabled" default="false" />
@@ -141,33 +143,10 @@
   <xacro:include filename="$(find udacity_bot)/urdf/rgb_camera.gazebo"/>
 </xacro:if>
-<!-- Laser -->
-<link name="hokuyo">
-    <pose>0 0 0.1 0 0 0</pose>
-    <inertial>
-      <mass value="0.1"/>
-      <origin xyz="0.0 0 0" rpy="0 0 0"/>
-      <inertia
-          ixx="0.0001" ixy="0" ixz="0"
-          iyy="0.0001" iyz="0"
-          izz="0.0001"
-      />
-    </inertial>
-    <collision name='hokuyo_collision'>
-      <origin xyz="0.0 0 0" rpy="0 0 0"/>
-      <geometry>
-        <box size="0.1 0.1 0.1"/>
-      </geometry>
-    </collision>
-    <visual name='hokuyo_visual'>
-      <origin xyz="0.0 0 0" rpy="0 0 0"/>
-      <geometry>
-         <mesh filename="package://udacity_bot/meshes/hokuyo.dae"/>
-      </geometry>
-    </visual>
-  </link>
-<joint type="fixed" name="hokuyo_joint">
-    <origin xyz="0.135 0 0.09" rpy="0 0 0"/> <!-- 0.15 -->
-    <child link="hokuyo"/>
-    <parent link="chassis"/>
-  </joint>
+<!-- Add a Hokuyo laser scanner -->
+<xacro:if value="$(arg add_laser_sensor)">
+  <!-- Add Laser link, joints and mesh -->
+  <xacro:include filename="$(find udacity_bot)/urdf/hokuyo_laser.xacro"/>
+  <!-- Add Gazebo Laser Plugin -->
+  <xacro:include filename="$(find udacity_bot)/urdf/hokuyo_laser.gazebo"/>
+</xacro:if>
 </robot>
